File: Overkeyboard.kicad_pcb (KiCad board)
At the start: 2 copper layers, 324 parts, among them SW1 SW_Push, SW10 SW_Push, SW100 SW_Push, SW101 SW_Push, SW102 SW_Push, SW103 SW_Push, SW104 SW_Push, SW105 SW_Push, SW106 SW_Push, SW107 SW_Push, SW108 SW_Push, SW109 SW_Push, SW11 SW_Push, SW110 SW_Push, SW111 SW_Push, SW112 SW_Push, SW113 SW_Push, SW114 SW_Push, SW115 SW_Push, SW116 SW_Push, SW117 SW_Push, SW118 SW_Push, SW119 SW_Push, SW12 SW_Push, SW120 SW_Push, SW121 SW_Push, SW122 SW_Push, SW123 SW_Push, SW124 SW_Push, SW125 SW_Push, SW126 SW_Push, SW127 SW_Push, SW128 SW_Push, SW129 SW_Push, SW13 SW_Push, SW130 SW_Push, SW131 SW_Push, SW132 SW_Push, SW133 SW_Push, SW134 SW_Push, SW135 SW_Push, SW136 SW_Push, SW137 SW_Push, SW138 SW_Push, SW139 SW_Push, SW14 SW_Push, SW140 SW_Push, SW141 SW_Push, SW142 SW_Push, SW143 SW_Push, SW144 SW_Push, SW145 SW_Push, SW146 SW_Push, SW147 SW_Push, SW148 SW_Push, SW149 SW_Push, SW15 SW_Push, SW150 SW_Push, SW151 SW_Push, SW152 SW_Push, SW153 SW_Push, SW154 SW_Push, SW155 SW_Push, SW156 SW_Push, SW157 SW_Push, SW16 SW_Push, SW17 SW_Push, SW18 SW_Push, SW19 SW_Push, SW2 SW_Push, SW20 SW_Push, SW21 SW_Push, SW22 SW_Push, SW23 SW_Push, SW24 SW_Push, SW25 SW_Push, SW26 SW_Push, SW27 SW_Push, SW28 SW_Push, SW29 SW_Push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

Commit message: It should be fully wired now
Parts:
- added C4: 0.1μF, Capacitor_SMD:C_0805_2012Metric_Pad1.18x1.45mm_HandSolder, B.Cu at (54.4, 74.4)
- added C5: 0.1μF, Capacitor_SMD:C_0805_2012Metric_Pad1.18x1.45mm_HandSolder, B.Cu at (42.5, 51.3)
- added C6: 0.1μF, Capacitor_SMD:C_0805_2012Metric_Pad1.18x1.45mm_HandSolder, B.Cu at (51.2, 51.4)
- added C7: 10μF, Capacitor_SMD:C_0805_2012Metric_Pad1.18x1.45mm_HandSolder, B.Cu at (58.5, 57.8)
- C1, C2, C3, D1, D10, D100, D101, D102, D103, D104, D105, D106, D107, D108, D109, D11, D110, D111, D112, D113, D114, D115, D116, D117, D118, D119, D12, D120, D121, D122, D123, D124, D125, D126, D127, D128, D129, D13, D130, D131, D132, D133, D134, D135, D136, D137, D138, D139, D14, D140, D141, D142, D143, D144, D145, D146, D147, D148, D149, D15, D151, D152, D153, D154, D155, D156, D157, D16, D17, D18, D19, D2, D20, D21, D22, D23, D24, D25, D26, D27, D28, D29, D3, D30, D31, D32, D33, D34, D35, D36, D37, D38, D39, D4, D40, D41, D42, D43, D44, D45, D46, D47, D48, D49, D5, D50, D51, D52, D53, D54, D55, D56, D57, D58, D59, D6, D60, D61, D62, D63, D64, D65, D66, D67, D68, D69, D7, D70, D71, D72, D73, D74, D75, D76, D77, D78, D79, D8, D80, D81, D82, D83, D84, D85, D86, D87, D88, D89, D9, D90, D91, D92, D93, D94, D95, D96, D97, D98, D99, F1, R1, R2, R3, R4, SW1, U1, USB1, Y1: moved to B.Cu
- SW146: footprint MX_Alps_Hybrid:MX-Alps-Hybrid-1U -> MX_Alps_Hybrid:MX-Alps-Hybrid-ISO
- SW81: footprint MX_Alps_Hybrid:MX-Alps-Hybrid-2U -> MX_Alps_Hybrid:MX-Alps-Hybrid-2U-Vertical
- moved D125 586.4 mm to (561.2, 41.3), turned to 90 degrees
- moved D126 579.0 mm to (561.2, 60.4), turned to 90 degrees
- moved D123 566.5 mm to (542.1, 41.3), turned to 90 degrees
- moved D124 559.0 mm to (542.1, 60.4), turned to 90 degrees
- moved D121 546.6 mm to (523.1, 41.3), turned to 90 degrees
- moved D133 546.1 mm to (561.2, 89.8), turned to 90 degrees
- moved D141 542.0 mm to (561.2, 127.9), turned to 90 degrees
- moved D134 540.5 mm to (561.2, 108.8), turned to 90 degrees
- moved D122 539.0 mm to (523.1, 60.4), turned to 90 degrees
- moved D142 536.7 mm to (561.2, 146.9), turned to 90 degrees
- moved D119 526.8 mm to (504.0, 41.3), turned to 90 degrees
- moved D131 525.9 mm to (542.1, 89.8), turned to 90 degrees
- moved D139 521.8 mm to (542.1, 127.9), turned to 90 degrees
- moved D132 520.3 mm to (542.1, 108.8), turned to 90 degrees
- moved D120 519.1 mm to (504.0, 60.4), turned to 90 degrees
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Connections:
- net +D renamed D+
- net -D renamed D-
- D101 pad 1: Net-(D101-K) -> ROW0
- D103 pad 1: Net-(D101-K) -> ROW0
- D105 pad 1: Net-(D101-K) -> ROW0
- D107 pad 1: Net-(D101-K) -> ROW0
- D109 pad 1: Net-(D101-K) -> ROW0
- D119 pad 1: Net-(D101-K) -> ROW0
- D121 pad 1: Net-(D101-K) -> ROW0
- D123 pad 1: Net-(D101-K) -> ROW0
- D125 pad 1: Net-(D101-K) -> ROW0
- D133 pad 2: unconnected-(D133-A-Pad2) -> Net-(D133-A)
- D134 pad 2: unconnected-(D134-A-Pad2) -> Net-(D134-A)
- D141 pad 2: unconnected-(D141-A-Pad2) -> Net-(D141-A)
- D142 pad 2: unconnected-(D142-A-Pad2) -> Net-(D142-A)
- D151 pad 1: Net-(D101-K) -> ROW0
- D7 pad 1: ROW5 -> ROW4
- D74 pad 1: unconnected-(D74-K-Pad1) -> ROW7
- D75 pad 1: unconnected-(D75-K-Pad1) -> ROW7
- D76 pad 1: unconnected-(D76-K-Pad1) -> ROW7
- D8 pad 1: ROW6 -> ROW5
- SW10 pad 1: Net-(D85-A) -> COL7
- SW10 pad 2: COL7 -> Net-(D85-A)
- SW100 pad 1: Net-(D15-A) -> COL3
- SW100 pad 2: COL3 -> Net-(D15-A)
- SW101 pad 1: Net-(D14-A) -> COL3
- SW101 pad 2: COL3 -> Net-(D14-A)
- SW102 pad 1: Net-(D18-A) -> COL4
- SW102 pad 2: COL4 -> Net-(D18-A)
- SW103 pad 1: Net-(D17-A) -> COL4
- SW103 pad 2: COL4 -> Net-(D17-A)
- SW104 pad 1: Net-(D41-A) -> COL4
- SW104 pad 2: COL4 -> Net-(D41-A)
- SW105 pad 1: Net-(D52-A) -> COL4
- SW105 pad 2: COL4 -> Net-(D52-A)
- SW106 pad 1: Net-(D19-A) -> COL5
- SW106 pad 2: COL5 -> Net-(D19-A)
- SW107 pad 1: Net-(D20-A) -> COL6
- SW107 pad 2: COL6 -> Net-(D20-A)
- SW108 pad 1: Net-(D21-A) -> COL7
- SW108 pad 2: COL7 -> Net-(D21-A)
- SW109 pad 1: Net-(D22-A) -> COL8
- SW109 pad 2: COL8 -> Net-(D22-A)
- SW11 pad 1: Net-(D86-A) -> COL7
- SW11 pad 2: COL7 -> Net-(D86-A)
- SW110 pad 1: Net-(D23-A) -> COL9
- SW110 pad 2: COL9 -> Net-(D23-A)
- SW111 pad 1: Net-(D24-A) -> COL10
- SW111 pad 2: COL10 -> Net-(D24-A)
- SW112 pad 1: Net-(D25-A) -> COL11
- SW112 pad 2: COL11 -> Net-(D25-A)
- SW113 pad 1: Net-(D26-A) -> COL12
- SW113 pad 2: COL12 -> Net-(D26-A)
- SW114 pad 1: Net-(D27-A) -> COL13
- SW114 pad 2: COL13 -> Net-(D27-A)
- SW115 pad 1: Net-(D28-A) -> COL14
- SW115 pad 2: COL14 -> Net-(D28-A)
- SW116 pad 1: Net-(D29-A) -> COL15
- SW116 pad 2: COL15 -> Net-(D29-A)
- SW117 pad 1: Net-(D30-A) -> COL16
- SW117 pad 2: COL16 -> Net-(D30-A)
- SW118 pad 1: Net-(D31-A) -> COL5
- SW118 pad 2: COL5 -> Net-(D31-A)
- SW119 pad 1: Net-(D32-A) -> COL6
- SW119 pad 2: COL6 -> Net-(D32-A)
- SW12 pad 1: Net-(D87-A) -> COL8
- SW12 pad 2: COL8 -> Net-(D87-A)
- SW120 pad 1: Net-(D33-A) -> COL7
- SW120 pad 2: COL7 -> Net-(D33-A)
- SW121 pad 1: Net-(D34-A) -> COL8
- SW121 pad 2: COL8 -> Net-(D34-A)
- SW122 pad 1: Net-(D35-A) -> COL9
- SW122 pad 2: COL9 -> Net-(D35-A)
- SW123 pad 1: Net-(D36-A) -> COL10
- SW123 pad 2: COL10 -> Net-(D36-A)
- SW124 pad 1: Net-(D37-A) -> COL11
- SW124 pad 2: COL11 -> Net-(D37-A)
- SW125 pad 1: Net-(D38-A) -> COL12
- SW125 pad 2: COL12 -> Net-(D38-A)
- SW126 pad 1: Net-(D39-A) -> COL13
- SW126 pad 2: COL13 -> Net-(D39-A)
- SW127 pad 1: Net-(D40-A) -> COL14
- SW127 pad 2: COL14 -> Net-(D40-A)
- SW128 pad 1: Net-(D42-A) -> COL5
- SW128 pad 2: COL5 -> Net-(D42-A)
- SW129 pad 1: Net-(D43-A) -> COL6
- SW129 pad 2: COL6 -> Net-(D43-A)
- SW13 pad 1: Net-(D88-A) -> COL8
- SW13 pad 2: COL8 -> Net-(D88-A)
- SW130 pad 1: Net-(D44-A) -> COL7
- SW130 pad 2: COL7 -> Net-(D44-A)
- SW131 pad 1: Net-(D45-A) -> COL8
- SW131 pad 2: COL8 -> Net-(D45-A)
- SW132 pad 1: Net-(D46-A) -> COL9
- SW132 pad 2: COL9 -> Net-(D46-A)
- SW133 pad 1: Net-(D47-A) -> COL10
- SW133 pad 2: COL10 -> Net-(D47-A)
- SW134 pad 1: Net-(D48-A) -> COL11
- SW134 pad 2: COL11 -> Net-(D48-A)
- SW135 pad 1: Net-(D49-A) -> COL12
- SW135 pad 2: COL12 -> Net-(D49-A)
- SW136 pad 1: Net-(D50-A) -> COL13
- SW136 pad 2: COL13 -> Net-(D50-A)
- SW137 pad 1: Net-(D53-A) -> COL5
- SW137 pad 2: COL5 -> Net-(D53-A)
- SW138 pad 1: Net-(D54-A) -> COL6
- SW138 pad 2: COL6 -> Net-(D54-A)
- SW139 pad 1: Net-(D55-A) -> COL7
- SW139 pad 2: COL7 -> Net-(D55-A)
- SW14 pad 1: Net-(D89-A) -> COL9
- SW14 pad 2: COL9 -> Net-(D89-A)
- SW140 pad 1: Net-(D56-A) -> COL8
- SW140 pad 2: COL8 -> Net-(D56-A)
- SW141 pad 1: Net-(D57-A) -> COL9
- SW141 pad 2: COL9 -> Net-(D57-A)
- SW142 pad 1: Net-(D58-A) -> COL10
- SW142 pad 2: COL10 -> Net-(D58-A)
- SW143 pad 1: Net-(D59-A) -> COL11
- SW143 pad 2: COL11 -> Net-(D59-A)
- SW144 pad 1: Net-(D60-A) -> COL12
- SW144 pad 2: COL12 -> Net-(D60-A)
- SW145 pad 1: Net-(D61-A) -> COL13
- SW145 pad 2: COL13 -> Net-(D61-A)
- SW146 pad 1: Net-(D51-A) -> COL16
- SW146 pad 2: COL16 -> Net-(D51-A)
- SW147 pad 1: Net-(D62-A) -> COL16
- SW147 pad 2: COL16 -> Net-(D62-A)
- SW148 pad 1: Net-(D64-A) -> COL11
- SW148 pad 2: COL11 -> Net-(D64-A)
- SW149 pad 1: Net-(D66-A) -> COL12
- SW149 pad 2: COL12 -> Net-(D66-A)
- SW15 pad 1: Net-(D90-A) -> COL9
- SW15 pad 2: COL9 -> Net-(D90-A)
- SW150 pad 1: Net-(D67-A) -> COL13
- SW150 pad 2: COL13 -> Net-(D67-A)
- SW151 pad 1: Net-(D70-A) -> COL16
- SW151 pad 2: COL16 -> Net-(D70-A)
- SW152 pad 1: Net-(D69-A) -> COL16
- SW152 pad 2: COL16 -> Net-(D69-A)
- SW153 pad 1: Net-(D68-A) -> COL12
- SW153 pad 2: COL13 -> Net-(D68-A)
- SW154 pad 1: Net-(D65-A) -> COL11
- SW154 pad 2: COL11 -> Net-(D65-A)
- SW155 pad 1: Net-(D63-A) -> COL7
- SW155 pad 2: COL7 -> Net-(D63-A)
- SW156 pad 1: Net-(D71-A) -> COL17
- SW156 pad 2: COL17 -> Net-(D71-A)
- SW157 pad 1: Net-(D72-A) -> COL17
- SW157 pad 2: COL17 -> Net-(D72-A)
- SW16 pad 1: Net-(D91-A) -> COL10
- SW16 pad 2: COL10 -> Net-(D91-A)
- SW17 pad 1: Net-(D92-A) -> COL10
- SW17 pad 2: COL10 -> Net-(D92-A)
- SW18 pad 1: Net-(D93-A) -> COL11
- SW18 pad 2: COL11 -> Net-(D93-A)
- SW19 pad 1: Net-(D94-A) -> COL11
- SW19 pad 2: COL11 -> Net-(D94-A)
- SW2 pad 1: Net-(D77-A) -> COL1
- SW2 pad 2: COL1 -> Net-(D77-A)
- SW20 pad 1: Net-(D95-A) -> COL13
- SW20 pad 2: COL13 -> Net-(D95-A)
- SW21 pad 1: Net-(D96-A) -> COL13
- SW21 pad 2: COL13 -> Net-(D96-A)
- SW22 pad 1: Net-(D97-A) -> COL14
- SW22 pad 2: COL14 -> Net-(D97-A)
- SW23 pad 1: Net-(D98-A) -> COL14
- SW23 pad 2: COL14 -> Net-(D98-A)
- SW24 pad 1: Net-(D99-A) -> COL15
- SW24 pad 2: COL15 -> Net-(D99-A)
- SW25 pad 1: Net-(D100-A) -> COL15
- SW25 pad 2: COL15 -> Net-(D100-A)
- SW26 pad 1: Net-(D101-A) -> COL16
- SW26 pad 2: COL16 -> Net-(D101-A)
- SW27 pad 1: Net-(D102-A) -> COL16
- SW27 pad 2: COL16 -> Net-(D102-A)
- SW28 pad 1: Net-(D103-A) -> COL17
- SW28 pad 2: COL17 -> Net-(D103-A)
- SW29 pad 1: Net-(D104-A) -> COL17
- SW29 pad 2: COL17 -> Net-(D104-A)
- SW3 pad 1: Net-(D78-A) -> COL1
- SW3 pad 2: COL1 -> Net-(D78-A)
- SW30 pad 1: Net-(D105-A) -> COL18
- SW30 pad 2: COL18 -> Net-(D105-A)
- SW31 pad 1: Net-(D106-A) -> COL18
- SW31 pad 2: COL18 -> Net-(D106-A)
- SW32 pad 1: Net-(D107-A) -> COL19
- SW32 pad 2: COL19 -> Net-(D107-A)
- SW33 pad 1: Net-(D108-A) -> COL19
- SW33 pad 2: COL19 -> Net-(D108-A)
- SW34 pad 1: Net-(D109-A) -> COL20
- SW34 pad 2: COL20 -> Net-(D109-A)
- SW35 pad 1: Net-(D110-A) -> COL20
- SW35 pad 2: COL20 -> Net-(D110-A)
- SW36 pad 1: Net-(D151-A) -> COL21
- SW36 pad 2: COL21 -> Net-(D151-A)
- SW37 pad 1: Net-(D152-A) -> COL21
- SW37 pad 2: COL21 -> Net-(D152-A)
- SW38 pad 1: Net-(D119-A) -> COL22
- SW38 pad 2: COL22 -> Net-(D119-A)
- SW39 pad 1: Net-(D120-A) -> COL22
- SW39 pad 2: COL22 -> Net-(D120-A)
- SW4 pad 1: Net-(D79-A) -> COL4
- SW4 pad 2: COL4 -> Net-(D79-A)
- SW40 pad 1: Net-(D121-A) -> COL23
- SW40 pad 2: COL23 -> Net-(D121-A)
- SW41 pad 1: Net-(D122-A) -> COL23
- SW41 pad 2: COL23 -> Net-(D122-A)
- SW42 pad 1: Net-(D123-A) -> COL24
- SW42 pad 2: COL24 -> Net-(D123-A)
- SW43 pad 1: Net-(D124-A) -> COL24
- SW43 pad 2: COL24 -> Net-(D124-A)
- SW44 pad 1: Net-(D125-A) -> COL25
- SW44 pad 2: COL25 -> Net-(D125-A)
- SW45 pad 1: Net-(D126-A) -> COL25
- SW45 pad 2: COL25 -> Net-(D126-A)
- SW46 pad 1: Net-(D111-A) -> COL17
- SW46 pad 2: COL17 -> Net-(D111-A)
- SW47 pad 1: Net-(D112-A) -> COL17
- SW47 pad 2: COL17 -> Net-(D112-A)
- SW48 pad 1: Net-(D113-A) -> COL18
- SW48 pad 2: COL18 -> Net-(D113-A)
- SW49 pad 1: Net-(D114-A) -> COL18
- SW49 pad 2: COL18 -> Net-(D114-A)
- SW5 pad 1: Net-(D80-A) -> COL4
- SW5 pad 2: COL4 -> Net-(D80-A)
- SW50 pad 1: Net-(D115-A) -> COL19
- SW50 pad 2: COL19 -> Net-(D115-A)
- SW51 pad 1: Net-(D116-A) -> COL19
- SW51 pad 2: COL19 -> Net-(D116-A)
- SW52 pad 1: Net-(D117-A) -> COL20
- SW52 pad 2: COL20 -> Net-(D117-A)
- SW53 pad 1: Net-(D118-A) -> COL20
- SW53 pad 2: COL20 -> Net-(D118-A)
- SW54 pad 1: Net-(D153-A) -> COL21
- SW54 pad 2: COL21 -> Net-(D153-A)
- SW55 pad 1: Net-(D154-A) -> COL21
- SW55 pad 2: COL21 -> Net-(D154-A)
- SW56 pad 1: Net-(D155-A) -> COL18
- SW56 pad 2: COL18 -> Net-(D155-A)
- SW57 pad 1: Net-(D156-A) -> COL19
- SW57 pad 2: COL19 -> Net-(D156-A)
- SW58 pad 1: Net-(D157-A) -> COL20
- SW58 pad 2: COL20 -> Net-(D157-A)
- SW59 pad 1: Net-(D127-A) -> COL22
- SW59 pad 2: COL22 -> Net-(D127-A)
- SW6 pad 1: Net-(D81-A) -> COL5
- SW6 pad 2: COL5 -> Net-(D81-A)
- SW60 pad 1: Net-(D128-A) -> COL22
- SW60 pad 2: COL22 -> Net-(D128-A)
- SW61 pad 1: Net-(D129-A) -> COL23
- SW61 pad 2: COL23 -> Net-(D129-A)
- SW62 pad 1: Net-(D130-A) -> COL23
- SW62 pad 2: COL23 -> Net-(D130-A)
- SW63 pad 1: Net-(D131-A) -> COL24
- SW63 pad 2: COL24 -> Net-(D131-A)
- SW64 pad 1: Net-(D132-A) -> COL24
- SW64 pad 2: COL24 -> Net-(D132-A)
- SW65 pad 1: unconnected-(SW65-Pad1) -> COL25
- SW65 pad 2: COL25 -> Net-(D133-A)
- SW66 pad 1: unconnected-(SW66-Pad1) -> COL25
- SW66 pad 2: COL25 -> Net-(D134-A)
- SW67 pad 1: Net-(D135-A) -> COL22
- SW67 pad 2: COL22 -> Net-(D135-A)
- SW68 pad 1: Net-(D136-A) -> COL22
- SW68 pad 2: COL22 -> Net-(D136-A)
- SW69 pad 1: Net-(D137-A) -> COL23
- SW69 pad 2: COL23 -> Net-(D137-A)
- SW7 pad 1: Net-(D82-A) -> COL5
- SW7 pad 2: COL5 -> Net-(D82-A)
- SW70 pad 1: Net-(D138-A) -> COL23
- SW70 pad 2: COL23 -> Net-(D138-A)
- SW71 pad 1: Net-(D139-A) -> COL24
- SW71 pad 2: COL24 -> Net-(D139-A)
- SW72 pad 1: Net-(D140-A) -> COL24
- SW72 pad 2: COL24 -> Net-(D140-A)
- SW73 pad 1: unconnected-(SW73-Pad1) -> COL25
- SW73 pad 2: COL25 -> Net-(D141-A)
- SW74 pad 1: unconnected-(SW74-Pad1) -> COL25
- SW74 pad 2: COL25 -> Net-(D142-A)
- SW75 pad 1: Net-(D143-A) -> COL22
- SW75 pad 2: COL22 -> Net-(D143-A)
- SW76 pad 1: Net-(D144-A) -> COL22
- SW76 pad 2: COL22 -> Net-(D144-A)
- SW77 pad 1: Net-(D145-A) -> COL23
- SW77 pad 2: COL23 -> Net-(D145-A)
- SW78 pad 1: Net-(D146-A) -> COL23
- SW78 pad 2: COL23 -> Net-(D146-A)
- SW79 pad 1: Net-(D147-A) -> COL24
- SW79 pad 2: COL24 -> Net-(D147-A)
- SW8 pad 1: Net-(D83-A) -> COL6
- SW8 pad 2: COL6 -> Net-(D83-A)
- SW80 pad 1: Net-(D148-A) -> COL24
- SW80 pad 2: COL24 -> Net-(D148-A)
- SW81 pad 1: Net-(D149-A) -> COL25
- SW81 pad 2: COL25 -> Net-(D149-A)
- SW82 pad 1: Net-(D74-A) -> COL18
- SW82 pad 2: COL18 -> Net-(D74-A)
- SW83 pad 1: Net-(D75-A) -> COL19
- SW83 pad 2: COL19 -> Net-(D75-A)
- SW84 pad 1: Net-(D76-A) -> COL20
- SW84 pad 2: COL20 -> Net-(D76-A)
- SW85 pad 1: Net-(D73-A) -> COL19
- SW85 pad 2: COL19 -> Net-(D73-A)
- SW86 pad 1: Net-(D1-A) -> COL1
- SW86 pad 2: COL1 -> Net-(D1-A)
- SW87 pad 1: Net-(D2-A) -> COL1
- SW87 pad 2: COL1 -> Net-(D2-A)
- SW88 pad 1: Net-(D3-A) -> COL1
- SW88 pad 2: COL1 -> Net-(D3-A)
- SW89 pad 1: Net-(D4-A) -> COL1
- SW89 pad 2: COL1 -> Net-(D4-A)
- SW9 pad 1: Net-(D84-A) -> COL6
- SW9 pad 2: COL6 -> Net-(D84-A)
- SW90 pad 1: Net-(D5-A) -> COL1
- SW90 pad 2: COL1 -> Net-(D5-A)
- SW91 pad 1: Net-(D6-A) -> COL1
- SW91 pad 2: COL1 -> Net-(D6-A)
- SW92 pad 1: Net-(D7-A) -> COL0
- SW92 pad 2: COL0 -> Net-(D7-A)
- SW93 pad 1: Net-(D8-A) -> COL0
- SW93 pad 2: COL0 -> Net-(D8-A)
- SW94 pad 1: Net-(D9-A) -> COL3
- SW94 pad 2: COL3 -> Net-(D9-A)
- SW95 pad 1: Net-(D10-A) -> COL3
- SW95 pad 2: COL3 -> Net-(D10-A)
- SW96 pad 1: Net-(D11-A) -> COL3
- SW96 pad 2: COL3 -> Net-(D11-A)
- SW97 pad 1: Net-(D12-A) -> COL2
- SW97 pad 2: COL2 -> Net-(D12-A)
- SW98 pad 1: Net-(D13-A) -> COL2
- SW98 pad 2: COL2 -> Net-(D13-A)
- SW99 pad 1: Net-(D16-A) -> COL3
- SW99 pad 2: COL3 -> Net-(D16-A)
- U1 pad 10: unconnected-(U1-PB0-Pad10) -> ROW1
- U1 pad 11: unconnected-(U1-PB1-Pad11) -> ROW2
- U1 pad 12: unconnected-(U1-PB2-Pad12) -> ROW3
- U1 pad 13: unconnected-(U1-PB3-Pad13) -> ROW4
- U1 pad 14: unconnected-(U1-PB4-Pad14) -> ROW5
- U1 pad 15: unconnected-(U1-PB5-Pad15) -> ROW6
- U1 pad 16: unconnected-(U1-PB6-Pad16) -> ROW7
- U1 pad 33: unconnected-(U1-PE0-Pad33) -> COL0
- U1 pad 34: unconnected-(U1-PE1-Pad34) -> COL1
- U1 pad 35: unconnected-(U1-PC0-Pad35) -> COL2
- U1 pad 36: unconnected-(U1-PC1-Pad36) -> COL3
- U1 pad 37: unconnected-(U1-PC2-Pad37) -> COL4
- U1 pad 38: unconnected-(U1-PC3-Pad38) -> COL5
- U1 pad 39: unconnected-(U1-PC4-Pad39) -> COL6
- U1 pad 40: unconnected-(U1-PC5-Pad40) -> COL7
- U1 pad 41: unconnected-(U1-PC6-Pad41) -> COL8
- U1 pad 42: unconnected-(U1-PC7-Pad42) -> COL9
- U1 pad 44: unconnected-(U1-PA7-Pad44) -> COL10
- U1 pad 45: unconnected-(U1-PA6-Pad45) -> COL11
- U1 pad 46: unconnected-(U1-PA5-Pad46) -> COL12
- U1 pad 47: unconnected-(U1-PA4-Pad47) -> COL13
- U1 pad 48: unconnected-(U1-PA3-Pad48) -> COL14
- U1 pad 49: unconnected-(U1-PA2-Pad49) -> COL15
- U1 pad 50: unconnected-(U1-PA1-Pad50) -> COL16
- U1 pad 51: unconnected-(U1-PA0-Pad51) -> COL17
- U1 pad 54: unconnected-(U1-PF7-Pad54) -> COL25
- U1 pad 55: unconnected-(U1-PF6-Pad55) -> COL24
- U1 pad 56: unconnected-(U1-PF5-Pad56) -> COL23
- U1 pad 57: unconnected-(U1-PF4-Pad57) -> COL22
- U1 pad 58: unconnected-(U1-PF3-Pad58) -> COL21
- U1 pad 59: unconnected-(U1-PF2-Pad59) -> COL20
- U1 pad 60: unconnected-(U1-PF1-Pad60) -> COL19
- U1 pad 61: unconnected-(U1-PF0-Pad61) -> COL18
- U1 pad 9: unconnected-(U1-PE3-Pad9) -> ROW0
- USB1 pad 5: unconnected-(USB1-VBUS-Pad5) -> VCC
- USB1 pad 6: VCC -> unconnected-(USB1-SHIELD-Pad6)
Routing:
- net ROW5: track 0.00 -> 708.6 mm
- net ROW6: track 0.00 -> 686.7 mm
- net COL25: track 0.00 -> 671.5 mm, vias 0 -> 1
- net COL24: track 0.00 -> 660.1 mm, vias 0 -> 1
- net ROW7: track 0.00 -> 655.7 mm
- net COL23: track 0.00 -> 639.1 mm, vias 0 -> 1
- net COL17: track 0.00 -> 637.4 mm, vias 0 -> 1
- net ROW4: track 0.00 -> 627.4 mm
- net COL14: track 0.00 -> 621.7 mm, vias 0 -> 1
- net COL22: track 0.00 -> 619.4 mm, vias 0 -> 1
- net COL16: track 0.00 -> 605.8 mm, vias 0 -> 1
- net COL15: track 0.00 -> 598.7 mm, vias 0 -> 1
- net ROW3: track 0.00 -> 590.8 mm
- net COL13: track 0.00 -> 589.3 mm, vias 0 -> 1
- net ROW0: track 0.00 -> 574.5 mm
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Other:
- board outline added: 555.6 x 198.4 mm
- board text added: "Do not draw traces past"

Commit message: Almost fully wired excepting figuring out what LED and resistor values to use
Parts:
- added D150: D_Small, Diode_SMD:D_SOD-123, B.Cu at (367.5, 108.7)
- added D158: LED, LED_THT:LED_D5.0mm, F.Cu at (176.2, 185.4)
- added D159: LED, LED_THT:LED_D5.0mm, F.Cu at (196.8, 185.4)
- added D160: LED, LED_THT:LED_D5.0mm, F.Cu at (217.5, 185.4)
- added D161: LED, LED_THT:LED_D5.0mm, F.Cu at (238.1, 185.4)
- added D162: LED, LED_THT:LED_D5.0mm, F.Cu at (258.8, 185.4)
- added R5: R_Small, Resistor_SMD:R_0805_2012Metric_Pad1.20x1.40mm_HandSolder, B.Cu at (176.2, 177.8)
- added R6: R_Small, Resistor_SMD:R_0805_2012Metric_Pad1.20x1.40mm_HandSolder, B.Cu at (196.8, 177.8)
- added R7: R_Small, Resistor_SMD:R_0805_2012Metric_Pad1.20x1.40mm_HandSolder, B.Cu at (217.5, 177.8)
- added R8: R_Small, Resistor_SMD:R_0805_2012Metric_Pad1.20x1.40mm_HandSolder, B.Cu at (238.1, 177.8)
- added R9: R_Small, Resistor_SMD:R_0805_2012Metric_Pad1.20x1.40mm_HandSolder, B.Cu at (258.8, 177.8)
- added SW158: SW_Push, MX_Solderable:MX-Solderable-1.5U, F.Cu at (358.0, 108.7)
- SW10, SW102, SW103, SW104, SW105, SW106, SW107, SW108, SW109, SW11, SW110, SW111, SW112, SW113, SW114, SW115, SW116, SW117, SW118, SW119, SW12, SW120, SW121, SW122, SW123, SW124, SW125, SW126, SW127, SW128, SW129, SW13, SW130, SW131, SW132, SW133, SW134, SW135, SW136, SW137, SW138, SW139, SW14, SW140, SW141, SW142, SW143, SW144, SW145, SW15, SW16, SW17, SW18, SW19, SW2, SW20, SW21, SW22, SW23, SW24, SW25, SW26, SW27, SW28, SW29, SW3, SW30, SW31, SW32, SW33, SW34, SW35, SW36, SW37, SW38, SW39, SW4, SW40, SW41, SW42, SW43, SW44, SW45, SW46, SW47, SW48, SW49, SW5, SW50, SW51, SW52, SW53, SW54, SW55, SW56, SW57, SW58, SW59, SW6, SW60, SW61, SW62, SW63, SW64, SW65, SW66, SW67, SW68, SW69, SW7, SW70, SW71, SW72, SW73, SW74, SW75, SW76, SW77, SW78, SW79, SW8, SW80, SW82, SW83, SW84, SW85, SW86, SW9, SW94, SW95, SW96, SW97, SW99: footprint MX_Alps_Hybrid:MX-Alps-Hybrid-1U -> MX_Solderable:MX-Solderable-1U
- SW100, SW148, SW149, SW150, SW151, SW154, SW156, SW157, SW89, SW90, SW92, SW93, SW98: footprint MX_Alps_Hybrid:MX-Alps-Hybrid-1.25U -> MX_Solderable:MX-Solderable-1.25U
- SW101, SW147, SW152, SW88: footprint MX_Alps_Hybrid:MX-Alps-Hybrid-1.75U -> MX_Solderable:MX-Solderable-1.75U
- SW146: footprint MX_Alps_Hybrid:MX-Alps-Hybrid-ISO -> MX_Solderable:MX-Solderable-2.25U
- SW153, SW91: footprint MX_Alps_Hybrid:MX-Alps-Hybrid-2U -> MX_Solderable:MX-Solderable-2U
- SW155: footprint MX_Alps_Hybrid:MX-Alps-Hybrid-6.25U -> MX_Solderable:MX-Solderable-6.25U
- SW81: footprint MX_Alps_Hybrid:MX-Alps-Hybrid-2U-Vertical -> MX_Solderable:MX-Solderable-2U-Vertical
- SW87: footprint MX_Alps_Hybrid:MX-Alps-Hybrid-1.5U -> MX_Solderable:MX-Solderable-1.5U
- moved USB1 20.1 mm to (79.7, 17.5)
- moved C1 20.1 mm to (78.5, 63.3)
- moved C3 20.1 mm to (67.4, 76.1)
- moved C4 20.1 mm to (74.5, 74.4)
- moved C6 20.1 mm to (71.3, 51.4)
- moved C2 20.1 mm to (57.6, 76.1)
- moved C5 20.1 mm to (62.6, 51.3)
- moved C7 20.1 mm to (78.6, 57.8)
- moved F1 20.1 mm to (74.1, 27.0)
- moved R1 20.1 mm to (62.7, 46.8)
- moved R2 20.1 mm to (81.2, 27.8)
- moved R3 20.1 mm to (78.1, 27.8)
- moved U1 20.1 mm to (65.8, 63.3)
- moved Y1 20.1 mm to (62.1, 76.1)
- moved R4 20.1 mm to (76.1, 77.6)
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Connections:
- U1 pad 28: unconnected-(U1-PD3-Pad28) -> LED0
- U1 pad 29: unconnected-(U1-PD4-Pad29) -> LED1
- U1 pad 30: unconnected-(U1-PD5-Pad30) -> LED2
- U1 pad 31: unconnected-(U1-PD6-Pad31) -> LED3
- U1 pad 32: unconnected-(U1-PD7-Pad32) -> LED4
- USB1 pad 6: unconnected-(USB1-SHIELD-Pad6) -> GND
Routing:
- net GND: track 171.5 -> 546.3 mm, vias 4 -> 6
- net LED4: track 0.00 -> 332.4 mm, vias 0 -> 1
- net LED3: track 0.00 -> 311.0 mm, vias 0 -> 1
- net LED2: track 0.00 -> 282.4 mm, vias 0 -> 1
- net LED1: track 0.00 -> 261.2 mm, vias 0 -> 1
- net LED0: track 0.00 -> 240.1 mm, vias 0 -> 1
- net ROW5: track 708.6 -> 672.2 mm
- net ROW4: track 627.4 -> 599.4 mm
- net +5V: track 105.2 -> 128.1 mm
- net COL22: track 619.4 -> 597.3 mm
- net COL21: track 511.6 -> 490.5 mm
- net COL24: track 660.1 -> 639.3 mm
- net COL19: track 545.6 -> 524.7 mm
- net COL18: track 524.6 -> 503.8 mm
- net COL23: track 639.1 -> 618.2 mm
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- added copper zone on B.Cu, net GND
Other:
- board size 555.6 x 198.4 mm -> 531.8 x 198.4 mm
- board text removed: "Do not draw traces past"

Commit message: slight wiring changes and LED resistor values determined
Parts:
- R1, R4: value 10k -> 10kΩ
- R2, R3: value 22 -> 22Ω
- R5, R6, R7, R8, R9: value R_Small -> 100Ω
Changed lines of the file:
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@@
 			(layer "F.SilkS"
 				(type "Top Silk Screen")
+				(color "White")
 			)
 			(layer "F.Paste"
@@
 			(layer "B.SilkS"
 				(type "Bottom Silk Screen")
+				(color "White")
 			)
 			(copper_finish "None")
@@
 		(tags "LED diameter 5.0mm 2 pins")
 		(property "Reference" "D158"
-			(at 1.27 -3.96 270)
+			(at 1.27 -3.96 -90)
 			(layer "F.SilkS")
 			(effects
@@
 		)
 		(property "Value" "LED"
-			(at 1.27 3.96 270)
+			(at 1.27 3.96 -90)
 			(layer "F.Fab")
 			(effects
@@
 		)
 		(fp_text user "${REFERENCE}"
-			(at 1.25 0 270)
+			(at 1.25 0 -90)
 			(layer "F.Fab")
 			(effects
@@
 		(tags "LED diameter 5.0mm 2 pins")
 		(property "Reference" "D161"
-			(at 1.27 -3.96 270)
+			(at 1.27 -3.96 -90)
 			(layer "F.SilkS")
 			(effects
@@
 		)
 		(property "Value" "LED"
-			(at 1.27 3.96 270)
+			(at 1.27 3.96 -90)
 			(layer "F.Fab")
 			(effects
@@
 		)
 		(fp_text user "${REFERENCE}"
-			(at 1.25 0 270)
+			(at 1.25 0 -90)
 			(layer "F.Fab")
 			(effects
@@
 		(tags "LED diameter 5.0mm 2 pins")
 		(property "Reference" "D160"
-			(at 1.27 -3.96 270)
+			(at 1.27 -3.96 -90)
 			(layer "F.SilkS")
 			(effects
@@
 		)
 		(property "Value" "LED"
-			(at 1.27 3.96 270)
+			(at 1.27 3.96 -90)
 			(layer "F.Fab")
 			(effects
@@
 		)
 		(fp_text user "${REFERENCE}"
-			(at 1.25 0 270)
+			(at 1.25 0 -90)
 			(layer "F.Fab")
 			(effects
@@
 		(tags "LED diameter 5.0mm 2 pins")
 		(property "Reference" "D159"
-			(at 1.27 -3.96 270)
+			(at 1.27 -3.96 -90)
 			(layer "F.SilkS")
 			(effects
@@
 		)
 		(property "Value" "LED"
-			(at 1.27 3.96 270)
+			(at 1.27 3.96 -90)
 			(layer "F.Fab")
 			(effects
@@
 		)
 		(fp_text user "${REFERENCE}"
-			(at 1.25 0 270)
+			(at 1.25 0 -90)
 			(layer "F.Fab")
 			(effects
@@
 		(tags "LED diameter 5.0mm 2 pins")
 		(property "Reference" "D162"
-			(at 1.27 -3.96 270)
+			(at 1.27 -3.96 -90)
 			(layer "F.SilkS")
 			(effects
@@
 		)
 		(property "Value" "LED"
-			(at 1.27 3.96 270)
+			(at 1.27 3.96 -90)
 			(layer "F.Fab")
 			(effects
@@
 		)
 		(fp_text user "${REFERENCE}"
-			(at 1.25 0 270)
+			(at 1.25 0 -90)
 			(layer "F.Fab")
 			(effects
@@
 			)
 		)
-		(property "Value" "R_Small"
+		(property "Value" "100Ω"
 			(at 0 -1.65 90)
 			(layer "B.Fab")
@@
 			)
 		)
-		(property "Value" "R_Small"
+		(property "Value" "100Ω"
 			(at 0 -1.65 90)
 			(layer "B.Fab")
@@
 			)
 		)
-		(property "Value" "R_Small"
+		(property "Value" "100Ω"
 			(at 0 -1.65 90)
 			(layer "B.Fab")
@@
 			)
 		)
-		(property "Value" "10k"
+		(property "Value" "10kΩ"
 			(at 0 -1.65 0)
 			(layer "B.Fab")
@@
 			)
 		)
-		(property "Value" "R_Small"
+		(property "Value" "100Ω"
 			(at 0 -1.65 90)
 			(layer "B.Fab")
@@
 			)
 		)
-		(property "Value" "R_Small"
+		(property "Value" "100Ω"
 			(at 0 -1.65 90)
 			(layer "B.Fab")
@@
 			)
 		)
-		(property "Value" "10k"
+		(property "Value" "10kΩ"
 			(at 0 -1.65 0)
 			(layer "B.Fab")
@@
 			)
 		)
-		(property "Value" "22"
+		(property "Value" "22Ω"
 			(at 0 -1.65 90)
 			(layer "B.Fab")
@@
 			)
 		)
-		(property "Value" "22"
+		(property "Value" "22Ω"
 			(at 0 -1.65 90)
 			(layer "B.Fab")

Commit message: fix some minor positional differences
Parts:
- moved D103 0.17 mm to (399.4, 41.3)
- moved D104 0.17 mm to (399.4, 60.3)
- moved D105 0.17 mm to (418.5, 41.3)
- moved D106 0.17 mm to (418.5, 60.3)
- moved D107 0.17 mm to (437.5, 41.3)
- moved D108 0.17 mm to (437.5, 60.3)
- moved D109 0.17 mm to (456.6, 41.3)
- moved D110 0.17 mm to (456.6, 60.3)
- moved D151 0.17 mm to (475.6, 41.3)
- moved D152 0.17 mm to (475.6, 60.3)
- moved SW28 0.17 mm to (391.3, 41.3)
- moved SW29 0.17 mm to (391.3, 60.3)
- moved SW30 0.17 mm to (410.4, 41.3)
- moved SW31 0.17 mm to (410.4, 60.3)
- moved SW32 0.17 mm to (429.4, 41.3)
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Routing:
- net GND: track 546.3 -> 542.7 mm
